File: hardware/pcb/pid2_levitador.sch (EAGLE design)
At the start: 160 parts, among them P1_C1 1u, P1_C2 1u, P1_C3 10n (opc.), P1_D1 1N5408, P1_D2 1N4148, P1_IC1 TL074CN, P1_IC2 TL074CN, P1_JP_GND GND-PGND, P1_J_COIL BOBINA, P1_J_IN VSENSOR, P1_J_OUT VPID, P1_J_PWR PWR, P1_J_VBOB VBOB, P1_POT1 22k, P1_POT2 220k, P1_POT3 22k, P1_POT4 10k, P1_Q1 TIP122, P1_R1 10k, P1_R10 1k, P1_R11 1M, P1_R12 160k, P1_R13 240k, P1_R14 96k, P1_R15 160k, P1_R16 270, P1_R17 56k, P1_R18 1k, P1_R2 10k, P1_R3 10k, P1_R4 10k, P1_R5 10k, P1_R6 1k, P1_R7 10k, P1_R8 10k, P1_R9 10k, P1_RBASE 270, P1_RBIAS 4.4k, P1_ROFFSET 10k, P1_RS 10 x 1R 5W, P2_C1 1u, P2_C2 1u, P2_C3 10n (opc.), P2_D1 1N5408, P2_D2 1N4148, P2_IC1 TL074CN, P2_IC2 TL074CN, P2_JP_GND GND-PGND, P2_J_COIL BOBINA, P2_J_IN VSENSOR, P2_J_OUT VPID, P2_J_PWR PWR, P2_J_VBOB VBOB, P2_POT1 22k, P2_POT2 220k, P2_POT3 22k, P2_POT4 10k, P2_Q1 TIP122, P2_R1 10k, P2_R10 1k, P2_R11 1M, P2_R12 160k, P2_R13 240k, P2_R14 96k, P2_R15 160k, P2_R16 270, P2_R17 56k, P2_R18 1k, P2_R2 10k, P2_R3 10k, P2_R4 10k, P2_R5 10k, P2_R6 1k, P2_R7 10k, P2_R8 10k, P2_R9 10k, P2_RBASE 270, P2_RBIAS 4.4k, P2_ROFFSET 10k, P2_RS 10 x 1R 5W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

Commit message: Placa de 2 PID por tarjeta (170 x 117 mm, cabe en 20 x 20 cm): banco de sensado de 3 x 1 ohm, R17 = 10 kohm, hojas de cobre y de ensamble con nombres U1 a U8
Parts:
- removed P3_C1, P3_C2, P4_C1, P4_C2: 1u, pid4:C
- removed P3_C3, P4_C3: 10n (opc.), pid4:C
- removed P3_D1, P4_D1: 1N5408, pid4:D1N5408
- removed P3_D2, P4_D2: 1N4148, pid4:D1N4148
- removed P3_IC1, P3_IC2, P4_IC1, P4_IC2: TL074CN, pid4:TL074
- removed P3_JP_GND, P4_JP_GND: GND-PGND, pid4:HDR2
- removed P3_J_COIL, P4_J_COIL: BOBINA, pid4:TERM2
- removed P3_J_IN, P4_J_IN: VSENSOR, pid4:HDR1
- removed P3_J_OUT, P4_J_OUT: VPID, pid4:HDR1
- removed P3_J_PWR, P4_J_PWR: PWR, pid4:HDR4
- removed P3_J_VBOB, P4_J_VBOB: VBOB, pid4:TERM2
- removed P3_POT1, P3_POT3, P4_POT1, P4_POT3: 22k, pid4:POT
- removed P3_POT2, P4_POT2: 220k, pid4:POT
- removed P3_POT4, P4_POT4: 10k, pid4:POT
- removed P3_Q1, P4_Q1: TIP122, pid4:TIP122
- removed P3_R1, P3_R2, P3_R3, P3_R4, P3_R5, P3_R7, P3_R8, P3_R9, P3_ROFFSET, P4_R1, P4_R2, P4_R3, P4_R4, P4_R5, P4_R7, P4_R8, P4_R9, P4_ROFFSET: 10k, pid4:R
- removed P3_R10, P3_R18, P3_R6, P4_R10, P4_R18, P4_R6: 1k, pid4:R
- removed P3_R11, P4_R11: 1M, pid4:R
- removed P3_R12, P3_R15, P4_R12, P4_R15: 160k, pid4:R
- removed P3_R13, P4_R13: 240k, pid4:R
- removed P3_R14, P4_R14: 96k, pid4:R
- removed P3_R16, P3_RBASE, P4_R16, P4_RBASE: 270, pid4:R
- removed P3_R17, P4_R17: 56k, pid4:R
- removed P3_RBIAS, P4_RBIAS: 4.4k, pid4:R
- removed P3_RS, P4_RS: 10 x 1R 5W, pid4:RSB
- P1_R17, P2_R17: value 56k -> 10k
- P1_RS, P2_RS: value 10 x 1R 5W -> 3 x 1R 5W
Connections:
- removed net P3_+VBOB: P3_D1.K, P3_J_COIL.1, P3_J_VBOB.1
- removed net P3_BASE: P3_D2.K, P3_Q1.B
- removed net P3_BASEA: P3_D2.A, P3_RBASE.2
- removed net P3_COILN: P3_D1.A, P3_J_COIL.2, P3_Q1.C
- removed net P3_INMU: P3_C3.1, P3_IC2D.IN-, P3_R18.2
- removed net P3_IOUT: P3_C3.2, P3_IC2D.OUT, P3_RBASE.1
- removed net P3_ISENSE: P3_Q1.E, P3_R18.1, P3_RS.1
- removed net P3_PGND: P3_JP_GND.2, P3_J_VBOB.2, P3_RS.2
- removed net P3_R6C2: P3_C2.1, P3_R6.2
- removed net P3_SUMN: P3_IC2B.IN-, P3_R10.1, P3_R7.2, P3_R8.2, P3_R9.2, P3_ROFFSET.2
- removed net P3_U1N: P3_IC1B.IN-, P3_R1.2, P3_R2.1
- removed net P3_U1P: P3_IC1B.IN+, P3_R3.2, P3_R4.1
- removed net P3_U2N: P3_IC1C.IN-, P3_POT1.1, P3_R5.2
- removed net P3_U3N: P3_C1.1, P3_IC1D.IN-, P3_POT2.2, P3_POT2.3, P3_R11.1
- removed net P3_U4N: P3_C2.2, P3_IC2A.IN-, P3_POT3.1
- removed net P3_U5P: P3_IC2B.IN+, P3_RBIAS.1
- removed net P3_VCAL: P3_POT4.2, P3_R16.1
- removed net P3_VD: P3_IC2A.OUT, P3_POT3.2, P3_POT3.3, P3_R9.1
- removed net P3_VDIV: P3_POT4.1, P3_R17.2
- removed net P3_VE: P3_IC1B.OUT, P3_POT2.1, P3_R2.2, P3_R5.1, P3_R6.1
- removed net P3_VI: P3_C1.2, P3_IC1D.OUT, P3_R11.2, P3_R8.1
- removed net P3_VINP: P3_IC2D.IN+, P3_R16.2
- removed net P3_VOFF: P3_IC2C.IN-, P3_IC2C.OUT, P3_ROFFSET.1
- removed net P3_VOFFD: P3_IC2C.IN+, P3_R14.2, P3_R15.1
- removed net P3_VP: P3_IC1C.OUT, P3_POT1.2, P3_POT1.3, P3_R7.1
- removed net P3_VPID: P3_IC2B.OUT, P3_J_OUT.1, P3_R10.2, P3_R17.1
- removed net P3_VREF: P3_IC1A.IN-, P3_IC1A.OUT, P3_R1.1
- removed net P3_VREFD: P3_IC1A.IN+, P3_R12.1, P3_R13.1
- removed net P3_VSEN: P3_J_IN.1, P3_R3.1
- removed net P4_+VBOB: P4_D1.K, P4_J_COIL.1, P4_J_VBOB.1
- removed net P4_BASE: P4_D2.K, P4_Q1.B
- removed net P4_BASEA: P4_D2.A, P4_RBASE.2
- removed net P4_COILN: P4_D1.A, P4_J_COIL.2, P4_Q1.C
- removed net P4_INMU: P4_C3.1, P4_IC2D.IN-, P4_R18.2
- removed net P4_IOUT: P4_C3.2, P4_IC2D.OUT, P4_RBASE.1
- removed net P4_ISENSE: P4_Q1.E, P4_R18.1, P4_RS.1
- removed net P4_PGND: P4_JP_GND.2, P4_J_VBOB.2, P4_RS.2
- removed net P4_R6C2: P4_C2.1, P4_R6.2
- removed net P4_SUMN: P4_IC2B.IN-, P4_R10.1, P4_R7.2, P4_R8.2, P4_R9.2, P4_ROFFSET.2
- removed net P4_U1N: P4_IC1B.IN-, P4_R1.2, P4_R2.1
- removed net P4_U1P: P4_IC1B.IN+, P4_R3.2, P4_R4.1
- removed net P4_U2N: P4_IC1C.IN-, P4_POT1.1, P4_R5.2
- removed net P4_U3N: P4_C1.1, P4_IC1D.IN-, P4_POT2.2, P4_POT2.3, P4_R11.1
- removed net P4_U4N: P4_C2.2, P4_IC2A.IN-, P4_POT3.1
- removed net P4_U5P: P4_IC2B.IN+, P4_RBIAS.1
- removed net P4_VCAL: P4_POT4.2, P4_R16.1
- removed net P4_VD: P4_IC2A.OUT, P4_POT3.2, P4_POT3.3, P4_R9.1
- removed net P4_VDIV: P4_POT4.1, P4_R17.2
- removed net P4_VE: P4_IC1B.OUT, P4_POT2.1, P4_R2.2, P4_R5.1, P4_R6.1
- removed net P4_VI: P4_C1.2, P4_IC1D.OUT, P4_R11.2, P4_R8.1
- removed net P4_VINP: P4_IC2D.IN+, P4_R16.2
- removed net P4_VOFF: P4_IC2C.IN-, P4_IC2C.OUT, P4_ROFFSET.1
- removed net P4_VOFFD: P4_IC2C.IN+, P4_R14.2, P4_R15.1
- removed net P4_VP: P4_IC1C.OUT, P4_POT1.2, P4_POT1.3, P4_R7.1
- removed net P4_VPID: P4_IC2B.OUT, P4_J_OUT.1, P4_R10.2, P4_R17.1
- removed net P4_VREF: P4_IC1A.IN-, P4_IC1A.OUT, P4_R1.1
- removed net P4_VREFD: P4_IC1A.IN+, P4_R12.1, P4_R13.1
- removed net P4_VSEN: P4_J_IN.1, P4_R3.1
- net +16V: no longer P3_IC1P.V+, P3_IC2P.V+, P3_J_PWR.1, P4_IC1P.V+, P4_IC2P.V+, P4_J_PWR.1
- net +5V: no longer P3_J_PWR.4, P3_R13.2, P4_J_PWR.4, P4_R13.2
- net -16V: no longer P3_IC1P.V-, P3_IC2P.V-, P3_J_PWR.2, P3_R14.1, P4_IC1P.V-, P4_IC2P.V-, P4_J_PWR.2, P4_R14.1
- net GND: no longer P3_IC1C.IN+, P3_IC1D.IN+, P3_IC2A.IN+, P3_JP_GND.1, P3_J_PWR.3, P3_POT4.3, P3_R12.2, P3_R15.2, P3_R4.2, P3_RBIAS.2, P4_IC1C.IN+, P4_IC1D.IN+, P4_IC2A.IN+, P4_JP_GND.1, P4_J_PWR.3, P4_POT4.3, P4_R12.2, P4_R15.2, P4_R4.2, P4_RBIAS.2
Other:
- note removed: "Módulo PID 3: controlador PID analógico (2 x TL074CN)"
- note removed: "Módulo PID 4: controlador PID analógico (2 x TL074CN)"
