File: fuente/hardware/pcb/fuente.sch (EAGLE design)
At the start: 57 parts, among them J1 SEC 18V, J2 SALIDA, J3 TP, Q1 TIP32C, Q2 BC557, Q3 TIP31C, Q4 BC547, U1 LM317T, U2 LM337T, U3 LM317T

Commit message: Fuente: C1 y C2 de 6800 uF/50 V (D28 mm, paso 10 mm) y F2 lento T1A
- Huella de C1/C2 ampliada a 28 mm de diámetro y taladro de 1.3 mm;
  se regeneran .brd/.sch, cobre espejado 1:1 y ensamble (sin cambios de ruteo).
- Cálculos, simulación, esquemáticos, informe, lista de materiales y
  tabla de mediciones actualizados (rizado del filtro 0.73/0.59 V pp).
Parts:
- C1, C2: value 3300u/50V -> 6800u/50V
- F2: value 1A 5x20 -> T1A 5x20
Changed lines of the file:
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@@
 <parts>
 <part name="J1" library="fuente16" deviceset="TERM2" device="" value="SEC 18V"/>
-<part name="F2" library="fuente16" deviceset="FUSE" device="" value="1A 5x20"/>
+<part name="F2" library="fuente16" deviceset="FUSE" device="" value="T1A 5x20"/>
 <part name="D1" library="fuente16" deviceset="D41" device="" value="1N4007"/>
 <part name="D2" library="fuente16" deviceset="D41" device="" value="1N4007"/>
-<part name="C1" library="fuente16" deviceset="CPOL25" device="" value="3300u/50V"/>
-<part name="C2" library="fuente16" deviceset="CPOL25" device="" value="3300u/50V"/>
+<part name="C1" library="fuente16" deviceset="CPOL25" device="" value="6800u/50V"/>
+<part name="C2" library="fuente16" deviceset="CPOL25" device="" value="6800u/50V"/>
 <part name="RSC1" library="fuente16" deviceset="R1W" device="" value="1R8 1W"/>
 <part name="RSC2" library="fuente16" deviceset="R1W" device="" value="2R2 1W"/>

Commit message: Fuente v2: ±16 V a 1,5 A con ampliación de corriente y foldback
- Transformador 18-0-18 V / 3 A con puente (onda completa); C1 15000 µF y 2x6800 µF reutilizados
- Limitador con foldback (Darlington TIP42C/BD140, sensor BC557) antes de cada regulador
- Ampliación de corriente (Fig. 3-21) con los mismos LM317/LM337
- Carga de prueba RL removible en J4/J5
- Cálculos, simulación (curva V-I, arranque con RL), esquemáticos, placa 190,5 x 139,7 mm,
  lista de materiales, plan de pruebas e informe actualizados
Parts:
- removed C2: 6800u/50V, fuente16:CPOL25
- added C18: 10u tant, fuente16:CTANT
- added C19, C3, C4: 100n, fuente16:C
- added C2A, C2B: 6800u/50V, fuente16:CPOL25
- added D12: 1N4148, fuente16:D35
- added D13: 1N4007, fuente16:D41
- added F3: T3.15A, fuente16:FUSE
- added J4: RL +16, fuente16:TERM2
- added J5: RL -16, fuente16:TERM2
- added Q5, Q8: TIP41C, fuente16:TIP41C
- added Q6: BD139, fuente16:BD139
- added Q7: BC547, fuente16:BC547
- added R15: 2R7 1W, fuente16:R1W
- added R16, R20: 120 1%, fuente16:R10
- added R17: 1k3 1%, fuente16:R10
- added R18: 2k2, fuente16:R10
- added R19: 100 3W, fuente16:R3W
- added R21: 330 1%, fuente16:R10
- added R22: 470, fuente16:R10
- C1: value 6800u/50V -> 15000u/50V; device fuente16:CPOL25 -> fuente16:CPOL35
- C11: value 10u tant -> 10u/25V; device fuente16:CTANT -> fuente16:CPOL5
- C12: value 100n -> 10u tant; device fuente16:C -> fuente16:CTANT
- C13: value 100u/25V -> 100n; device fuente16:CPOL6 -> fuente16:C
- C14: value 100n -> 220u/25V; device fuente16:C -> fuente16:CPOL8
- C15: value 10u/25V -> 100u/25V; device fuente16:CPOL5 -> fuente16:CPOL6
- C16: value 10u tant -> 100n; device fuente16:CTANT -> fuente16:C
- C17, C6: value 100n -> 10u/25V; device fuente16:C -> fuente16:CPOL5
- C7: value 10u/25V -> 10u tant; device fuente16:CPOL5 -> fuente16:CTANT
- C8: value 10u/25V -> 100n; device fuente16:CPOL5 -> fuente16:C
- C9: value 10u tant -> 220u/25V; device fuente16:CTANT -> fuente16:CPOL8
- D1, D2, D3, D7: value 1N4007 -> 1N5408; device fuente16:D41 -> fuente16:D201
- D10, D4: value 1N4148 -> 1N5408; device fuente16:D35 -> fuente16:D201
- D9: value 1N4007 -> 1N4148; device fuente16:D41 -> fuente16:D35
- F2: value T1A 5x20 -> T3.15A
- J1: value SEC 18V -> SEC 18-0-18; device fuente16:TERM2 -> fuente16:TERM3
- Q1: value TIP32C -> TIP42C; device fuente16:TIP32C -> fuente16:TIP42C
- Q2: value BC557 -> BD140; device fuente16:BC557 -> fuente16:BD140
- Q3: value TIP31C -> BC557; device fuente16:TIP31C -> fuente16:BC557
- Q4: value BC547 -> TIP42C; device fuente16:BC547 -> fuente16:TIP42C
- R10: value 120 1% -> 2k2
- R11: value 330 1% -> 2k7 1W; device fuente16:R10 -> fuente16:R1W
- R12: value 2k2 -> 1k
- R13: value 2k2 -> 270
- R14: value 470 -> 12k
- R3: value 820 2W -> 2k7 1W; device fuente16:R2W -> fuente16:R1W
- R4: value 820 2W -> 1k; device fuente16:R2W -> fuente16:R10
- R5: value 120 1% -> 270
- R6: value 120 1% -> 12k
- R7: value 1k3 1% -> 2R7 1W; device fuente16:R10 -> fuente16:R1W
- R8: value 1k3 1% -> 120 1%
- R9: value 100 3W -> 1k3 1%; device fuente16:R3W -> fuente16:R10
- RSC1: value 1R8 1W -> 0R27 5W; device fuente16:R1W -> fuente16:R5W
- RSC2: value 2R2 1W -> 0R27 5W; device fuente16:R1W -> fuente16:R5W
Connections:
- removed net AC: D1.A, D2.K, F2.2
- removed net ACIN: F2.1, J1.2
- removed net LED2A: LED2.A, R13.2
- removed net VB1: Q1.B, Q2.C, R3.1
- removed net VB3: Q3.B, Q4.C, R4.1
- removed net VE1: Q1.E, Q2.B, RSC1.2
- removed net VE3: Q3.E, Q4.B, RSC2.2
- removed net VIN1: C5.1, D3.K, Q1.C, U1.IN
- removed net VIN2: C6.2, D5.A, Q3.C, U2.IN
- new net AC1: D1.A, D3.K, F2.2
- new net AC2: D2.A, D4.K, F3.2
- new net ACA: F2.1, J1.1
- new net ACB: F3.1, J1.3
- new net B1: Q1.B, Q2.E, R4.2
- new net B2: Q5.B, Q6.E, R12.2
- new net BD1: Q2.B, Q3.C, R3.1
- new net BD2: Q6.B, Q7.C, R11.1
- new net BS1: Q3.B, R5.1, R6.1
- new net BS2: Q7.B, R13.1, R14.1
- new net E1: Q1.E, R4.1, R5.2, RSC1.2
- new net E2: Q5.E, R12.1, R13.2, RSC2.2
- new net IN1: C5.1, D5.K, Q4.B, R7.2, U1.IN
- new net IN2: C10.2, D8.A, Q8.B, R15.2, U2.IN
- new net LED2K: LED2.K, R18.2
- new net VA1: Q1.C, Q2.C, Q4.E, R6.2, R7.1
- new net VA2: Q5.C, Q6.C, Q8.E, R14.2, R15.1
- net +16V: now also C7.+, C8.1, D5.A, D6.K, J4.1, Q4.C, R10.1, R19.1, R8.1; no longer C10.1, D3.A, D4.K, R12.1, R5.1, R9.1
- net +5V: now also C18.+, C19.1, D11.A, D12.K, D13.K, R20.1, R22.1; no longer C16.+, C17.1, D10.K, D11.K, D9.A, R10.1, R14.1
- net -16V: now also C12.-, C13.2, C14.-, D10.A, D8.K, D9.A, J5.1, Q8.C, R16.1, R18.1; no longer C11.-, C12.2, D5.K, D6.A, D8.A, LED2.K, R6.1
- net ADJ1: now also C6.+, D6.A, R8.2, R9.1; no longer C7.+, D4.A, R5.2, R7.1
- net ADJ2: now also C11.-, D9.K, R16.2, R17.1; no longer C8.-, D6.K, R6.2, R8.1
- net ADJ3: now also C17.+, D12.A, R20.2, R21.1; no longer C15.+, D10.A, R10.2, R11.1
- net GND: now also C10.1, C12.+, C13.1, C14.+, C16.2, C17.-, C18.-, C19.2, C2A.+, C2B.+, C3.2, C4.1, C6.-, C8.2, D10.K, D13.A, J1.2, J4.2, J5.2, LED2.A, R11.2; no longer C10.2, C12.1, C13.-, C14.2, C16.-, C17.2, C2.+, C6.1, C8.+, D11.A, D8.K, J1.1, R13.1, R4.2
- net LED1A: now also R10.2; no longer R12.2
- net LED3A: now also R22.2; no longer R14.2
- net RV1A: now also R9.2; no longer R7.2
- net RV2A: now also R17.2; no longer R8.2
- net RV3A: now also R21.2; no longer R11.2
- net VIN3: now also C15.+, C16.1, D11.K, R19.2; no longer C13.+, C14.1, D9.K, R9.2
- net VRAWN: now also C2A.-, C2B.-, C4.2, D3.A, D4.A, Q7.E; no longer C2.-, D2.A, Q4.E
- net VRAWP: now also C3.1, D2.K, Q3.E; no longer Q2.E
Other:
- note added: "Ampliación y regulador +16 V"
- note added: "Ampliación y regulador -16 V"
- note added: "Entrada, puente y filtros"
- note added: "Filtro - y puntos de prueba"
- note added: "Fuente ±16 V / 1,5 A y +5 V, versión 2 (conexiones por etiquetas de red; ver esquematicos/ para el dibujo)"
- note added: "Limitador +16 V (foldback)"
- note added: "Limitador -16 V (foldback)"
- note removed: "Entrada y rectificadores"
- note removed: "Fuente ±16 V / +5 V para los 4 PID del levitador (conexiones por etiquetas de red; ver esquematicos/ para el dibujo)"
- note removed: "Limitador +16 V"
- note removed: "Limitador -16 V"
- note removed: "Regulador +16 V"
- note removed: "Regulador -16 V"
- moved on the sheet: C1, C10, C11, C15, C5, C7, C9, D1, D10, D11, D2, D3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
